Commit message: Fixed bug in wheel xacro macro. Fixed bug in base_link origin tags

File: urdf/diff_drive_4.urdf.xacro (robot description, xacro)
@@ -1,4 +1,8 @@
 <?xml version="1.0"?>
 <robot name="roscontrol" xmlns:xacro="http://ros.org/wiki/xacro">
+  <!--
+    Run the following command to check if the urdf file is ok:
+    ~$ xacro diff_drive_4.urdf.xacro > tmp.urdf && check_urdf tmp.urdf && rm tmp.urdf
+  -->
   <!-- Xacro properties definition -->
   <xacro:property name="odom_dist_wh" value="0.2"/>
@@ -59,5 +63,5 @@
       <!-- axis and rotation always defined relative to parent frame -->
       <axis xyz="0 1 0" rpy="0 0 0" />
-      <parent link="${base_link}"/>
+      <parent link="base_link"/>
       <child link="${prefix}_${suffix}_wheel"/>
       <origin xyz="${offset} ${reflect*odom_dist_wh/2} 0" rpy="0 0 0"/>
@@ -88,7 +92,7 @@
   <link name="base_link">
     <visual>
+      <origin xyz="${odom_diam/2-body_len/2} 0 ${-odom_diam/2+body_gnd_height+body_height/2}"
+              rpy="0 0 0"/>
       <geometry>
-        <origin xyz="${odom_diam/2-body_len/2} 0 ${-odom_diam/2+body_gnd_height+body_height/2}"
-                rpy="0 0 0"/>
         <box size="${body_len} ${body_width} ${body_height}"/>
       </geometry>
@@ -96,7 +100,7 @@
     </visual>
     <collision>
+      <origin xyz="${odom_diam/2-body_len/2} 0 ${-odom_diam/2+body_gnd_height+body_height/2}"
+              rpy="0 0 0"/>
       <geometry>
-        <origin xyz="${odom_diam/2-body_len/2} 0 ${-odom_diam/2+body_gnd_height+body_height/2}"
-                rpy="0 0 0"/>
         <box size="${body_len} ${body_width} ${body_height}"/>
       </geometry>

Commit message: Changed length of the robot's body

File: urdf/diff_drive_4.urdf.xacro (robot description, xacro)
@@ -14,5 +14,5 @@
   <xacro:property name="body_gnd_height" value="0.02"/>
   <xacro:property name="body_wh_space" value="0.005"/>
-  <xacro:property name="body_len" value="0.6"/>
+  <xacro:property name="body_len" value="0.3"/>
   <xacro:property name="body_width"
                   value="${odom_dist_wh-wh_thick-2*body_wh_space}"/>

Commit message: Fixed inertia models of the 4-wh diff drive Bug detected when the robot is rotating around itself. Problem due odom reference frame being wrongly defined.

File: urdf/diff_drive_4.urdf.xacro (robot description, xacro)
@@ -29,11 +29,6 @@
   </material>
   <!-- Xacro Macro definitions -->
-  <!-- + default inertial model (dependent on the objects mass): -->
-  <xacro:macro name="default_inertial" params="mass">
-    <inertial>
-      <mass value="${mass}"/>
-      <inertia ixx="1.0" ixy="0.0" ixz="0.0" iyy="1.0" iyz="0.0" izz="1.0"/>
-    </inertial>
-  </xacro:macro>
+  <!-- + inertial models: -->
+  <xacro:include filename="inertia.urdf.xacro"/>
   <!-- + wheel macro:
          - prefix  : relative to the default name
@@ -58,5 +53,6 @@
         </geometry>
       </collision>
-      <xacro:default_inertial mass="0.05"/>
+      <xacro:inertial_wh_cylinder mass="0.05"
+                                  radius="${odom_diam/2}" height="${wh_thick}"/>
     </link>
     <joint name="${prefix}_${suffix}_wheel_joint" type="continuous">
@@ -106,5 +102,7 @@
       </geometry>
     </collision>
-    <xacro:default_inertial mass="1.00"/>
+    <xacro:inertial_body_cuboid mass="1.00"
+                                size_x="${body_len}" size_y="${body_width}"
+                                size_z="${body_height}"/>
   </link>
   <!-- Wheels -->

Commit message: Fixed bug on odom reference frame The problem of rotating around its center is solved. Another bug is reported for the cmd_vel/angular/z.

File: urdf/diff_drive_4.urdf.xacro (robot description, xacro)
@@ -88,5 +88,5 @@
   <link name="base_link">
     <visual>
-      <origin xyz="${odom_diam/2-body_len/2} 0 ${-odom_diam/2+body_gnd_height+body_height/2}"
+      <origin xyz="0 0 ${-odom_diam/2+body_gnd_height+body_height/2}"
               rpy="0 0 0"/>
       <geometry>
@@ -96,5 +96,5 @@
     </visual>
     <collision>
-      <origin xyz="${odom_diam/2-body_len/2} 0 ${-odom_diam/2+body_gnd_height+body_height/2}"
+      <origin xyz="0 0 ${-odom_diam/2+body_gnd_height+body_height/2}"
               rpy="0 0 0"/>
       <geometry>
@@ -107,10 +107,12 @@
   </link>
   <!-- Wheels -->
-  <xacro:wheel prefix="right" suffix="front" reflect="-1"/>
-  <xacro:wheel prefix="left"  suffix="front" reflect="1"/>
+  <xacro:wheel prefix="right" suffix="front" reflect="-1"
+               offset="${body_len/2-odom_diam/2}"/>
+  <xacro:wheel prefix="left"  suffix="front" reflect="1"
+               offset="${body_len/2-odom_diam/2}"/>
   <xacro:wheel prefix="right" suffix="back"  reflect="-1"
-               offset="${odom_diam-body_len}"/>
+               offset="-${body_len/2-odom_diam/2}"/>
   <xacro:wheel prefix="left"  suffix="back"  reflect="1"
-               offset="${odom_diam-body_len}"/>
+               offset="-${body_len/2-odom_diam/2}"/>
   <!-- Gazebo plugin for ROS Control -->
   <gazebo>
