Commit message: Version 0.1.2: Laser 2D on top of the robots

File: urdf/diff_drive.urdf.xacro (robot description, xacro)
@@ -31,5 +31,6 @@
   <!-- Xacro Macro definitions -->
   <!-- + inertial models: -->
-  <xacro:include filename="inertia.urdf.xacro"/>
+  <xacro:include
+    filename="$(find robot_sim_diff_drive_rbs)/urdf/inertia.urdf.xacro"/>
   <!-- + caster wheel macro: -->
   <xacro:macro name="caster_wheel" params="prefix reflect">
@@ -152,4 +153,12 @@
   <xacro:caster_wheel prefix="front" reflect="1"/>
   <xacro:caster_wheel prefix="back"  reflect="-1"/>
+  <!-- Sensors -->
+  <xacro:include
+      filename="$(find robot_sim_diff_drive_rbs)/urdf/hokuyo_ust10.urdf.xacro"/>
+  <xacro:hokuyo_ust10_mount prefix="base" topic="base_laser"
+                            parent_link="base_link">
+    <origin xyz="0 0 ${-odom_diam/2+body_gnd_height+body_height}"
+            rpy="0 0 0"/>
+  </xacro:hokuyo_ust10_mount>
   <!-- Gazebo plugin for ROS Control -->
   <gazebo>

File: urdf/diff_drive_4.urdf.xacro (robot description, xacro)
@@ -30,5 +30,6 @@
   <!-- Xacro Macro definitions -->
   <!-- + inertial models: -->
-  <xacro:include filename="inertia.urdf.xacro"/>
+  <xacro:include
+    filename="$(find robot_sim_diff_drive_rbs)/urdf/inertia.urdf.xacro"/>
   <!-- + wheel macro:
          - prefix  : relative to the default name
@@ -116,4 +117,12 @@
   <xacro:wheel prefix="left"  suffix="back"  reflect="1"
                offset="-${body_len/2-odom_diam/2}"/>
+  <!-- Sensors -->
+  <xacro:include
+      filename="$(find robot_sim_diff_drive_rbs)/urdf/hokuyo_ust10.urdf.xacro"/>
+  <xacro:hokuyo_ust10_mount prefix="base" topic="base_laser"
+                            parent_link="base_link">
+    <origin xyz="0 0 ${-odom_diam/2+body_gnd_height+body_height}"
+            rpy="0 0 0"/>
+  </xacro:hokuyo_ust10_mount>
   <!-- Gazebo plugin for ROS Control -->
   <gazebo>

Commit message: Model compatible with different radius for each wheel

File: urdf/diff_drive.urdf.xacro (robot description, xacro)
@@ -7,8 +7,10 @@
   <!-- Xacro properties definition -->
   <xacro:property name="odom_dist_wh" value="0.2"/>
-  <xacro:property name="odom_diam_wh_r" value="0.06"/>
-  <xacro:property name="odom_diam_wh_l" value="0.06"/>
+  <xacro:property name="odom_diam_wh_r" value="0.07"/>
+  <xacro:property name="odom_diam_wh_l" value="0.05"/>
   <xacro:property name="odom_diam"
                   value="${(odom_diam_wh_r+odom_diam_wh_l)/2}"/>
+  <xacro:property name="odom_diam_max"
+                  value="${max(odom_diam_wh_r,odom_diam_wh_l)}"/>
   <xacro:property name="wh_thick" value="0.005"/>
   <xacro:property name="wh_caster_diam" value="0.01"/>
@@ -62,5 +64,5 @@
       <child link="${prefix}_caster_wheel"/>
       <origin
-        xyz="${reflect*(body_len/2-wh_caster_diam/2)} 0 ${wh_caster_diam/2-odom_diam/2}"
+        xyz="${reflect*(body_len/2-wh_caster_diam/2)} 0 ${wh_caster_diam/2-odom_diam_max/2}"
         rpy="0 0 0"/>
     </joint>
@@ -73,9 +75,10 @@
   </xacro:macro>
   <!-- + wheel macro:
+         - diameter: diameter of the wheel
          - prefix  : relative to the default name
          - reflect : 1 or -1 (default or inverted orientation relative to
                      parent frame)
          - offset  : relative to the parent frame in x axis -->
-  <xacro:macro name="wheel" params="prefix reflect offset:=0">
+  <xacro:macro name="wheel" params="diameter prefix reflect offset:=0">
     <link name="${prefix}_wheel">
       <visual>
@@ -83,5 +86,5 @@
         <origin xyz="0 0 0" rpy="${pi/2} 0 0" />
         <geometry>
-          <cylinder radius="${odom_diam/2}" length="${wh_thick}"/>
+          <cylinder radius="${diameter/2}" length="${wh_thick}"/>
         </geometry>
         <material name="black"/>
@@ -90,9 +93,9 @@
         <origin xyz="0 0 0" rpy="${pi/2} 0 0" />
         <geometry>
-          <cylinder radius="${odom_diam/2}" length="${wh_thick}"/>
+          <cylinder radius="${diameter/2}" length="${wh_thick}"/>
         </geometry>
       </collision>
       <xacro:inertial_wh_cylinder mass="0.05"
-                                  radius="${odom_diam/2}" height="${wh_thick}"/>
+                                  radius="${diameter/2}" height="${wh_thick}"/>
     </link>
     <joint name="${prefix}_wheel_joint" type="continuous">
@@ -129,5 +132,5 @@
   <link name="base_link">
     <visual>
-      <origin xyz="0 0 ${-odom_diam/2+body_gnd_height+body_height/2}"
+      <origin xyz="0 0 ${-odom_diam_max/2+body_gnd_height+body_height/2}"
               rpy="0 0 0"/>
       <geometry>
@@ -137,5 +140,5 @@
     </visual>
     <collision>
-      <origin xyz="0 0 ${-odom_diam/2+body_gnd_height+body_height/2}"
+      <origin xyz="0 0 ${-odom_diam_max/2+body_gnd_height+body_height/2}"
               rpy="0 0 0"/>
       <geometry>
@@ -148,6 +151,6 @@
   </link>
   <!-- Wheels -->
-  <xacro:wheel prefix="right" reflect="-1" offset="0"/>
-  <xacro:wheel prefix="left"  reflect="1"  offset="0"/>
+  <xacro:wheel diameter="${odom_diam_wh_r}" prefix="right" reflect="-1"/>
+  <xacro:wheel diameter="${odom_diam_wh_l}" prefix="left"  reflect="1"/>
   <!-- Caster Wheels -->
   <xacro:caster_wheel prefix="front" reflect="1"/>
@@ -158,5 +161,5 @@
   <xacro:hokuyo_ust10_mount prefix="base" topic="base_laser"
                             parent_link="base_link">
-    <origin xyz="0 0 ${-odom_diam/2+body_gnd_height+body_height}"
+    <origin xyz="0 0 ${-odom_diam_max/2+body_gnd_height+body_height}"
             rpy="0 0 0"/>
   </xacro:hokuyo_ust10_mount>

Commit message: Changed collision and visual of base_link

File: urdf/diff_drive.urdf.xacro (robot description, xacro)
@@ -132,5 +132,6 @@
   <link name="base_link">
     <visual>
-      <origin xyz="0 0 ${-odom_diam_max/2+body_gnd_height+body_height/2}"
+      <origin
+        xyz="${odom_diam_max/2-body_len/2} 0 ${-odom_diam_max/2+body_gnd_height+body_height/2}"
               rpy="0 0 0"/>
       <geometry>
@@ -143,9 +144,9 @@
               rpy="0 0 0"/>
       <geometry>
-        <box size="${body_len} ${body_width} ${body_height}"/>
+        <box size="${odom_diam_max} ${body_width} ${body_height}"/>
       </geometry>
     </collision>
     <xacro:inertial_body_cuboid mass="1.00"
-                                size_x="${body_len}" size_y="${body_width}"
+                                size_x="${odom_diam_max}" size_y="${body_width}"
                                 size_z="${body_height}"/>
   </link>

Commit message: Fixed gravity bug for diff_drive with a laser

File: urdf/diff_drive.urdf.xacro (robot description, xacro)
@@ -7,6 +7,6 @@
   <!-- Xacro properties definition -->
   <xacro:property name="odom_dist_wh" value="0.2"/>
-  <xacro:property name="odom_diam_wh_r" value="0.07"/>
-  <xacro:property name="odom_diam_wh_l" value="0.05"/>
+  <xacro:property name="odom_diam_wh_r" value="0.06"/>
+  <xacro:property name="odom_diam_wh_l" value="0.06"/>
   <xacro:property name="odom_diam"
                   value="${(odom_diam_wh_r+odom_diam_wh_l)/2}"/>
@@ -21,4 +21,11 @@
                   value="${odom_dist_wh-wh_thick-2*body_wh_space}"/>
   <xacro:property name="body_height" value="0.1"/>
+  <xacro:property name="laser_lx" value="0.0"/>
+  <xacro:property name="laser_ly" value="0.0"/>
+  <xacro:property name="laser_lz"
+                  value="${-odom_diam_max/2+body_gnd_height+body_height}"/>
+  <xacro:property name="laser_rr" value="0.0"/>
+  <xacro:property name="laser_rp" value="0.0"/>
+  <xacro:property name="laser_ry" value="0.0"/>
   <!-- Materials definition -->
   <material name="blue">
@@ -36,5 +43,5 @@
     filename="$(find robot_sim_diff_drive_rbs)/urdf/inertia.urdf.xacro"/>
   <!-- + caster wheel macro: -->
-  <xacro:macro name="caster_wheel" params="prefix reflect">
+  <xacro:macro name="caster_wheel" params="prefix reflect offset:=0">
     <link name="${prefix}_caster_wheel">
       <visual>
@@ -64,5 +71,5 @@
       <child link="${prefix}_caster_wheel"/>
       <origin
-        xyz="${reflect*(body_len/2-wh_caster_diam/2)} 0 ${wh_caster_diam/2-odom_diam_max/2}"
+        xyz="${reflect*offset} 0 ${wh_caster_diam/2-odom_diam_max/2}"
         rpy="0 0 0"/>
     </joint>
@@ -141,13 +148,13 @@
     </visual>
     <collision>
-      <origin xyz="0 0 ${-odom_diam_max/2+body_gnd_height+body_height/2}"
-              rpy="0 0 0"/>
+      <origin
+        xyz="${odom_diam_max/2-body_len/2} 0 ${-odom_diam_max/2+body_gnd_height+body_height/2}"
+        rpy="0 0 0"/>
       <geometry>
-        <box size="${odom_diam_max} ${body_width} ${body_height}"/>
+        <box size="${body_len} ${body_width} ${body_height}"/>
       </geometry>
     </collision>
-    <xacro:inertial_body_cuboid mass="1.00"
-                                size_x="${odom_diam_max}" size_y="${body_width}"
-                                size_z="${body_height}"/>
+    <xacro:inertial_body_cuboid mass="1.00" size_x="${body_len}"
+                                size_y="${body_width}" size_z="${body_height}"/>
   </link>
   <!-- Wheels -->
@@ -155,6 +162,6 @@
   <xacro:wheel diameter="${odom_diam_wh_l}" prefix="left"  reflect="1"/>
   <!-- Caster Wheels -->
-  <xacro:caster_wheel prefix="front" reflect="1"/>
-  <xacro:caster_wheel prefix="back"  reflect="-1"/>
+  <xacro:caster_wheel prefix="back" reflect="-1"
+                      offset="${body_len-odom_diam_max}"/>
   <!-- Sensors -->
   <xacro:include
@@ -162,6 +169,6 @@
   <xacro:hokuyo_ust10_mount prefix="base" topic="base_laser"
                             parent_link="base_link">
-    <origin xyz="0 0 ${-odom_diam_max/2+body_gnd_height+body_height}"
-            rpy="0 0 0"/>
+    <origin xyz="${laser_lx} ${laser_ly} ${laser_lz}"
+            rpy="${laser_rr} ${laser_rp} ${laser_ry}"/>
   </xacro:hokuyo_ust10_mount>
   <!-- Gazebo plugin for ROS Control -->

File: urdf/hokuyo_ust10.urdf.xacro (robot description, xacro)
@@ -15,5 +15,5 @@
       </link-->
       <gazebo reference="${frame}">
-        <turnGravityOff>true</turnGravityOff>
+        <turnGravityOff>false</turnGravityOff>
         <sensor type="ray" name="${frame}">
           <pose>0 0 0 0 0 0</pose>
